Commit message: parameter tuning

File: fennec_description/urdf/fennec.xacro (robot description, xacro)
@@ -56,4 +56,12 @@
   </link>
   <!-- Front steer and rear wheel joints required for ackermann_steering_controller -->
+  <xacro:rear_wheel
+    name="rear"
+    parent="base"
+    wheel_radius="${wheel_radius/4}"
+    wheel_thickness="${wheel_thickness/2}"
+    wheel_mass="${wheel_mass/32}">
+    <origin xyz="${-base_length/2+axle_offset} 0 0" rpy="${-90 * deg_to_rad} 0 0"/>
+  </xacro:rear_wheel>
   <xacro:front_steer
     name="front"
@@ -67,12 +75,21 @@
     steer_height="${wheel_radius+steer_offset}">
   </xacro:front_steer>
-  <xacro:rear_wheel
-    name="rear"
+  <!-- Rear wheels -->
+  <xacro:rear_wheel_lr
+    name="rear_right"
     parent="base"
-    wheel_radius="${wheel_radius/4}"
-    wheel_thickness="${wheel_thickness/2}"
-    wheel_mass="${wheel_mass/32}">
-    <origin xyz="${-base_length/2+axle_offset} 0 0" rpy="${-90 * deg_to_rad} 0 0"/>
-  </xacro:rear_wheel>
+    wheel_radius="${wheel_radius}"
+    wheel_thickness="${wheel_thickness}"
+    wheel_mass="${wheel_mass}">
+    <origin xyz="${-base_length/2+axle_offset} ${-base_width/2-axle_offset} 0" rpy="${-90 * deg_to_rad} 0 0"/>
+  </xacro:rear_wheel_lr>
+  <xacro:rear_wheel_lr
+    name="rear_left"
+    parent="base"
+    wheel_radius="${wheel_radius}"
+    wheel_thickness="${wheel_thickness}"
+    wheel_mass="${wheel_mass}">
+    <origin xyz="${-base_length/2+axle_offset} ${+base_width/2+axle_offset} 0" rpy="${-90 * deg_to_rad} 0 0"/>
+  </xacro:rear_wheel_lr>
   <!-- Steerable front wheels -->
   <xacro:front_wheel_lr
@@ -106,21 +123,4 @@
     steer_height="${wheel_radius+steer_offset}">
   </xacro:front_wheel_lr>
-  <!-- Rear wheels -->
-  <xacro:rear_wheel_lr
-    name="rear_right"
-    parent="base"
-    wheel_radius="${wheel_radius}"
-    wheel_thickness="${wheel_thickness}"
-    wheel_mass="${wheel_mass}">
-    <origin xyz="${-base_length/2+axle_offset} ${-base_width/2-axle_offset} 0" rpy="${-90 * deg_to_rad} 0 0"/>
-  </xacro:rear_wheel_lr>
-  <xacro:rear_wheel_lr
-    name="rear_left"
-    parent="base"
-    wheel_radius="${wheel_radius}"
-    wheel_thickness="${wheel_thickness}"
-    wheel_mass="${wheel_mass}">
-    <origin xyz="${-base_length/2+axle_offset} ${+base_width/2+axle_offset} 0" rpy="${-90 * deg_to_rad} 0 0"/>
-  </xacro:rear_wheel_lr>
   <!-- Colour -->
   <gazebo reference="base_link">

File: fennec_description/urdf/wheel.xacro (robot description, xacro)
@@ -11,4 +11,141 @@
   <xacro:property name="steer_velocity" value="5.0"/>
   <xacro:property name="steer_limit_deg" value="45.0"/>
+  <!-- Bicycle model rear wheel link (required for steer_drive_controller) -->
+  <xacro:macro name="rear_wheel"
+    params="
+      name
+      parent
+      wheel_radius
+      wheel_thickness
+      wheel_mass
+      *origin">
+    <link name="${name}_wheel_link">
+      <visual>
+        <origin xyz="0 0 0" rpy="0 0 0"/>
+        <geometry>
+          <cylinder radius="${wheel_radius}" length="${wheel_thickness}"/>
+        </geometry>
+        <material name="yellow" />
+      </visual>
+      <collision>
+        <origin xyz="0 0 0" rpy="0 0 0"/>
+        <geometry>
+          <cylinder radius="${wheel_radius}" length="${wheel_thickness}"/>
+        </geometry>
+      </collision>
+      <xacro:solid_cylinder_inertial
+          rpy="0 0 0" xyz="0 0 0"
+          mass="${wheel_mass}"
+          radius="${wheel_radius}" length="${wheel_thickness}" />
+    </link>
+    <joint name="${name}_wheel_joint" type="continuous">
+      <parent link="${parent}_link"/>
+      <child link="${name}_wheel_link"/>
+      <xacro:insert_block name="origin"/>
+      <axis xyz="0 0 1"/>
+    </joint>
+    <transmission name="${name}_wheel_joint_trans">
+      <type>transmission_interface/SimpleTransmission</type>
+      <actuator name="${name}_wheel_joint_motor">
+        <mechanicalReduction>1</mechanicalReduction>
+        <hardwareInterface>hardware_interface/VelocityJointInterface</hardwareInterface>
+      </actuator>
+      <joint name="${name}_wheel_joint">
+        <hardwareInterface>hardware_interface/VelocityJointInterface</hardwareInterface>
+      </joint>
+    </transmission>
+    <gazebo reference="${name}_wheel_link">
+      <material>Gazebo/Yellow</material>
+    </gazebo>
+  </xacro:macro>
+  <!-- Car steering model rear wheel links (left/right) -->
+  <xacro:macro name="rear_wheel_lr"
+    params="
+      name
+      parent
+      wheel_radius
+      wheel_thickness
+      wheel_mass
+      *origin">
+    <link name="${name}_wheel_link">
+      <visual>
+        <origin xyz="0 0 0" rpy="0 0 0"/>
+        <geometry>
+          <cylinder radius="${wheel_radius}" length="${wheel_thickness}"/>
+        </geometry>
+        <material name="red" />
+      </visual>
+      <collision>
+        <origin xyz="0 0 0" rpy="0 0 0"/>
+        <geometry>
+          <cylinder radius="${wheel_radius}" length="${wheel_thickness}"/>
+        </geometry>
+      </collision>
+      <xacro:solid_cylinder_inertial
+          rpy="0 0 0" xyz="0 0 0"
+          mass="${wheel_mass}"
+          radius="${wheel_radius}" length="${wheel_thickness}" />
+    </link>
+    <joint name="${name}_wheel_joint" type="continuous">
+      <parent link="${parent}_link"/>
+      <child link="${name}_wheel_link"/>
+      <xacro:insert_block name="origin"/>
+      <axis xyz="0 0 1"/>
+    </joint>
+    <transmission name="${name}_wheel_joint_trans">
+      <type>transmission_interface/SimpleTransmission</type>
+      <actuator name="${name}_wheel_joint_motor">
+        <mechanicalReduction>1</mechanicalReduction>
+        <hardwareInterface>hardware_interface/VelocityJointInterface</hardwareInterface>
+      </actuator>
+      <joint name="${name}_wheel_joint">
+        <hardwareInterface>hardware_interface/VelocityJointInterface</hardwareInterface>
+      </joint>
+    </transmission>
+    <gazebo reference="${name}_wheel_link">
+      <material>Gazebo/Red</material>
+    </gazebo>
+  </xacro:macro>
+  <!-- Bicycle model front wheel link (passive - no transmission) -->
+  <xacro:macro name="front_wheel"
+    params="
+      name
+      parent
+      wheel_radius
+      wheel_thickness
+      wheel_mass
+      *origin">
+    <link name="${name}_wheel_link">
+      <visual>
+        <origin xyz="0 0 0" rpy="0 0 0"/>
+        <geometry>
+          <cylinder radius="${wheel_radius}" length="${wheel_thickness}"/>
+        </geometry>
+        <material name="yellow" />
+      </visual>
+      <collision>
+        <origin xyz="0 0 0" rpy="0 0 0"/>
+        <geometry>
+          <cylinder radius="${wheel_radius}" length="${wheel_thickness}"/>
+        </geometry>
+      </collision>
+      <xacro:solid_cylinder_inertial
+          rpy="0 0 0" xyz="0 0 0"
+          mass="${wheel_mass}"
+          radius="${wheel_radius}" length="${wheel_thickness}" />
+    </link>
+    <joint name="${name}_wheel_joint" type="continuous">
+      <parent link="${parent}_link"/>
+      <child link="${name}_wheel_link"/>
+      <xacro:insert_block name="origin"/>
+      <axis xyz="0 0 1"/>
+    </joint>
+    <gazebo reference="${name}_wheel_link">
+      <material>Gazebo/Yellow</material>
+    </gazebo>
+    <gazebo reference="${name}_wheel_joint">
+      <provideFeedback>true</provideFeedback>
+    </gazebo>
+  </xacro:macro>
   <!-- Bicycle model front steering link (required for steer_drive_controller) -->
   <xacro:macro name="front_steer"
@@ -161,140 +298,3 @@
     </gazebo>
   </xacro:macro>
-  <!-- Bicycle model rear wheel link (required for steer_drive_controller) -->
-  <xacro:macro name="rear_wheel"
-    params="
-      name
-      parent
-      wheel_radius
-      wheel_thickness
-      wheel_mass
-      *origin">
-    <link name="${name}_wheel_link">
-      <visual>
-        <origin xyz="0 0 0" rpy="0 0 0"/>
-        <geometry>
-          <cylinder radius="${wheel_radius}" length="${wheel_thickness}"/>
-        </geometry>
-        <material name="yellow" />
-      </visual>
-      <collision>
-        <origin xyz="0 0 0" rpy="0 0 0"/>
-        <geometry>
-          <cylinder radius="${wheel_radius}" length="${wheel_thickness}"/>
-        </geometry>
-      </collision>
-      <xacro:solid_cylinder_inertial
-          rpy="0 0 0" xyz="0 0 0"
-          mass="${wheel_mass}"
-          radius="${wheel_radius}" length="${wheel_thickness}" />
-    </link>
-    <joint name="${name}_wheel_joint" type="continuous">
-      <parent link="${parent}_link"/>
-      <child link="${name}_wheel_link"/>
-      <xacro:insert_block name="origin"/>
-      <axis xyz="0 0 1"/>
-    </joint>
-    <transmission name="${name}_wheel_joint_trans">
-      <type>transmission_interface/SimpleTransmission</type>
-      <actuator name="${name}_wheel_joint_motor">
-        <mechanicalReduction>1</mechanicalReduction>
-        <hardwareInterface>hardware_interface/VelocityJointInterface</hardwareInterface>
-      </actuator>
-      <joint name="${name}_wheel_joint">
-        <hardwareInterface>hardware_interface/VelocityJointInterface</hardwareInterface>
-      </joint>
-    </transmission>
-    <gazebo reference="${name}_wheel_link">
-      <material>Gazebo/Yellow</material>
-    </gazebo>
-  </xacro:macro>
-  <!-- Bicycle model front wheel link (passive - no transmission) -->
-  <xacro:macro name="front_wheel"
-    params="
-      name
-      parent
-      wheel_radius
-      wheel_thickness
-      wheel_mass
-      *origin">
-    <link name="${name}_wheel_link">
-      <visual>
-        <origin xyz="0 0 0" rpy="0 0 0"/>
-        <geometry>
-          <cylinder radius="${wheel_radius}" length="${wheel_thickness}"/>
-        </geometry>
-        <material name="yellow" />
-      </visual>
-      <collision>
-        <origin xyz="0 0 0" rpy="0 0 0"/>
-        <geometry>
-          <cylinder radius="${wheel_radius}" length="${wheel_thickness}"/>
-        </geometry>
-      </collision>
-      <xacro:solid_cylinder_inertial
-          rpy="0 0 0" xyz="0 0 0"
-          mass="${wheel_mass}"
-          radius="${wheel_radius}" length="${wheel_thickness}" />
-    </link>
-    <joint name="${name}_wheel_joint" type="continuous">
-      <parent link="${parent}_link"/>
-      <child link="${name}_wheel_link"/>
-      <xacro:insert_block name="origin"/>
-      <axis xyz="0 0 1"/>
-    </joint>
-    <gazebo reference="${name}_wheel_link">
-      <material>Gazebo/Yellow</material>
-    </gazebo>
-    <gazebo reference="${name}_wheel_joint">
-      <provideFeedback>true</provideFeedback>
-    </gazebo>
-  </xacro:macro>
-  <!-- Car steering model rear wheel links (left/right) -->
-  <xacro:macro name="rear_wheel_lr"
-    params="
-      name
-      parent
-      wheel_radius
-      wheel_thickness
-      wheel_mass
-      *origin">
-    <link name="${name}_wheel_link">
-      <visual>
-        <origin xyz="0 0 0" rpy="0 0 0"/>
-        <geometry>
-          <cylinder radius="${wheel_radius}" length="${wheel_thickness}"/>
-        </geometry>
-        <material name="red" />
-      </visual>
-      <collision>
-        <origin xyz="0 0 0" rpy="0 0 0"/>
-        <geometry>
-          <cylinder radius="${wheel_radius}" length="${wheel_thickness}"/>
-        </geometry>
-      </collision>
-      <xacro:solid_cylinder_inertial
-          rpy="0 0 0" xyz="0 0 0"
-          mass="${wheel_mass}"
-          radius="${wheel_radius}" length="${wheel_thickness}" />
-    </link>
-    <joint name="${name}_wheel_joint" type="continuous">
-      <parent link="${parent}_link"/>
-      <child link="${name}_wheel_link"/>
-      <xacro:insert_block name="origin"/>
-      <axis xyz="0 0 1"/>
-    </joint>
-    <transmission name="${name}_wheel_joint_trans">
-      <type>transmission_interface/SimpleTransmission</type>
-      <actuator name="${name}_wheel_joint_motor">
-        <mechanicalReduction>1</mechanicalReduction>
-        <hardwareInterface>hardware_interface/VelocityJointInterface</hardwareInterface>
-      </actuator>
-      <joint name="${name}_wheel_joint">
-        <hardwareInterface>hardware_interface/VelocityJointInterface</hardwareInterface>
-      </joint>
-    </transmission>
-    <gazebo reference="${name}_wheel_link">
-      <material>Gazebo/Red</material>
-    </gazebo>
-  </xacro:macro>
 </robot>

Commit message: try replacing the urdf with a simpler one

File: fennec_description/urdf/fennec.xacro (robot description, xacro)
@@ -1,129 +1,108 @@
-<?xml version="1.0"?>
-<!--
-  Geometry:
-    The Ackermann steering controllers require the longitudinal
-    separation between the front and back wheel axes and the
-    lateral separation between the left and right front steering axes.
-    For this model:
-    wheel_separation_h = base_length - 2 * axle_offset = 0.4
-    wheel_separation_w = base_width  + 2 * axle_offset = 0.4
--->
-<robot name="fennec" xmlns:xacro="http://wiki.ros.org/xacro">
-  <!-- Include xacro for inertials, materials and wheels -->
-  <xacro:include filename="$(find fennec_description)/urdf/wheel.xacro"/>
-  <!-- Gazebo plugins -->
-  <gazebo>
-    <plugin name="gazebo_ros_control" filename="libgazebo_ros_control.so">
-    </plugin>
-  </gazebo>
-  <!-- Math constants -->
-  <xacro:property name="deg_to_rad" value="0.01745329251994329577"/>
-  <!-- Robot base dimensions -->
-  <xacro:property name="base_length" value="0.34" />
-  <xacro:property name="base_width" value="0.16" />
-  <xacro:property name="base_height" value="0.16" />
-  <xacro:property name="base_mass" value="5" />
-  <!-- Wheel link dimensions -->
-  <xacro:property name="wheel_radius" value="0.034" />
-  <xacro:property name="wheel_thickness" value="0.025" />
-  <xacro:property name="wheel_mass" value="1" />
-  <!-- Steering link dimensions -->
-  <xacro:property name="steer_radius" value="0.05" />
-  <xacro:property name="steer_thickness" value="0.02" />
-  <xacro:property name="steer_mass" value="1" />
-  <!-- Axle positions -->
-  <xacro:property name="axle_offset" value="0.035" />
-  <xacro:property name="steer_offset" value="0.01" />
-  <!-- Base link -->
-  <link name="base_link">
+<?xml version='1.0' ?>
+<robot name="jetracer" xmlns:xacro="http://www.ros.org/wiki/xacro">
+  <material name="black">
+    <color rgba="0 0 0 1"/>
+  </material>
+  <link name="base">
     <visual>
-      <origin xyz="0 0 0" rpy="0 0 0"/>
+      <orgin rpy="0 0 0" xyz="0 0 0"/>
       <geometry>
-        <box size="${base_length} ${base_width} ${base_height}"/>
+        <box size="1 2 0.3"/>
       </geometry>
-      <material name="green" />
     </visual>
-    <collision>
-      <origin xyz="0 0 0" rpy="0 0 0"/>
+  </link>
+  <!--Front left wheel-->
+  <joint name="fl_holder_joint" type="revolute">
+    <axis xyz="0 0 1"/>
+    <limit effort="1000.0" lower="-0.4" upper="0.4" velocity="0.5"/>
+    <origin rpy="0 0 0" xyz="-0.5 0.8 0"/>
+    <parent link="base"/>
+    <child link="fl_wheel_link"/>
+  </joint>
+  <link name="fl_wheel_link">
+    <visual>
+      <orgin rpy="0 0 0" xyz="-0.7 0.8 0"/>
       <geometry>
-        <box size="${base_length} ${base_width} ${base_height}"/>
+        <box size="0 0 0"/>
       </geometry>
-    </collision>
-    <xacro:solid_cuboid_inertial
-        rpy="0 0 0" xyz="0 0 0"
-        mass="${base_mass}"
-        x="${base_length}" y="${base_width}" z="${base_height}" />
+    </visual>
   </link>
-  <!-- Front steer and rear wheel joints required for ackermann_steering_controller -->
-  <xacro:rear_wheel
-    name="rear"
-    parent="base"
-    wheel_radius="${wheel_radius/4}"
-    wheel_thickness="${wheel_thickness/2}"
-    wheel_mass="${wheel_mass/32}">
-    <origin xyz="${-base_length/2+axle_offset} 0 0" rpy="${-90 * deg_to_rad} 0 0"/>
-  </xacro:rear_wheel>
-  <xacro:front_steer
-    name="front"
-    parent="base"
-    steer_radius="${steer_radius}"
-    steer_thickness="${steer_thickness}"
-    steer_mass="${steer_mass}"
-    base_length="${base_length}"
-    base_width="${base_width}"
-    axle_offset="${axle_offset}"
-    steer_height="${wheel_radius+steer_offset}">
-  </xacro:front_steer>
-  <!-- Rear wheels -->
-  <xacro:rear_wheel_lr
-    name="rear_right"
-    parent="base"
-    wheel_radius="${wheel_radius}"
-    wheel_thickness="${wheel_thickness}"
-    wheel_mass="${wheel_mass}">
-    <origin xyz="${-base_length/2+axle_offset} ${-base_width/2-axle_offset} 0" rpy="${-90 * deg_to_rad} 0 0"/>
-  </xacro:rear_wheel_lr>
-  <xacro:rear_wheel_lr
-    name="rear_left"
-    parent="base"
-    wheel_radius="${wheel_radius}"
-    wheel_thickness="${wheel_thickness}"
-    wheel_mass="${wheel_mass}">
-    <origin xyz="${-base_length/2+axle_offset} ${+base_width/2+axle_offset} 0" rpy="${-90 * deg_to_rad} 0 0"/>
-  </xacro:rear_wheel_lr>
-  <!-- Steerable front wheels -->
-  <xacro:front_wheel_lr
-    name="front_right"
-    parent="base"
-    reflect="-1"
-    wheel_radius="${wheel_radius}"
-    wheel_thickness="${wheel_thickness}"
-    wheel_mass="${wheel_mass}"
-    steer_radius="${steer_radius}"
-    steer_thickness="${steer_thickness}"
-    steer_mass="${steer_mass}"
-    base_length="${base_length}"
-    base_width="${base_width}"
-    axle_offset="${axle_offset}"
-    steer_height="${wheel_radius+steer_offset}">
-  </xacro:front_wheel_lr>
-  <xacro:front_wheel_lr
-    name="front_left"
-    parent="base"
-    reflect="1"
-    wheel_radius="${wheel_radius}"
-    wheel_thickness="${wheel_thickness}"
-    wheel_mass="${wheel_mass}"
-    steer_radius="${steer_radius}"
-    steer_thickness="${steer_thickness}"
-    steer_mass="${steer_mass}"
-    base_length="${base_length}"
-    base_width="${base_width}"
-    axle_offset="${axle_offset}"
-    steer_height="${wheel_radius+steer_offset}">
-  </xacro:front_wheel_lr>
-  <!-- Colour -->
-  <gazebo reference="base_link">
-    <material>Gazebo/Green</material>
-  </gazebo>
+  <joint name="fl_wheel_joint" type="continuous">
+    <axis xyz="0 0 1"/>
+    <origin rpy="0 1.57 0" xyz="-0.2 0 0"/>
+    <parent link="fl_wheel_link"/>
+    <child link="fl_wheel"/>
+  </joint>
+  <link name="fl_wheel">
+    <visual>
+      <orgin rpy="0 0 0" xyz="-0.7 0.8 0"/>
+      <geometry>
+        <cylinder radius="0.4" length="0.2"/>
+      </geometry>
+      <material name="black"/>
+    </visual>
+  </link>
+  <!--Front right wheel-->
+  <joint name="fr_holder_joint" type="revolute">
+    <axis xyz="0 0 1"/>
+    <limit effort="1000.0" lower="-0.4" upper="0.4" velocity="0.5"/>
+    <origin rpy="0 0 0" xyz="0.5 0.8 0"/>
+    <parent link="base"/>
+    <child link="fr_wheel_link"/>
+  </joint>
+  <link name="fr_wheel_link">
+    <visual>
+      <orgin rpy="0 0 0" xyz="0.7 0.8 0"/>
+      <geometry>
+        <box size="0 0 0"/>
+      </geometry>
+    </visual>
+  </link>
+  <joint name="fr_wheel_joint" type="continuous">
+    <axis xyz="0 0 1"/>
+    <origin rpy="0 1.57 0" xyz="0.2 0 0"/>
+    <parent link="fr_wheel_link"/>
+    <child link="fr_wheel"/>
+  </joint>
+  <link name="fr_wheel">
+    <visual>
+      <orgin rpy="0 0 0" xyz="0.7 0.8 0"/>
+      <geometry>
+        <cylinder radius="0.4" length="0.2"/>
+      </geometry>
+      <material name="black"/>
+    </visual>
+  </link>
+  <!--Rear left wheel-->
+  <joint name="rl_wheel_joint" type="continuous">
+    <axis xyz="0 0 1"/>
+    <origin rpy="0 1.57 0" xyz="-0.7 -0.8 0"/>
+    <parent link="base"/>
+    <child link="rl_wheel"/>
+  </joint>
+  <link name="rl_wheel">
+    <visual>
+      <orgin rpy="0 0 0" xyz="-0.7 -0.8 0"/>
+      <geometry>
+        <cylinder radius="0.4" length="0.2"/>
+      </geometry>
+      <material name="black"/>
+    </visual>
+  </link>
+  <!--Rear right wheel-->
+  <joint name="rr_wheel_joint" type="continuous">
+    <axis xyz="0 0 1"/>
+    <origin rpy="0 1.57 0" xyz="0.7 -0.8 0"/>
+    <parent link="base"/>
+    <child link="rr_wheel"/>
+  </joint>
+  <link name="rr_wheel">
+    <visual>
+      <orgin rpy="0 0 0" xyz="0.7 -0.8 0"/>
+      <geometry>
+        <cylinder radius="0.4" length="0.2"/>
+      </geometry>
+      <material name="black"/>
+    </visual>
+  </link>
 </robot>
