Commit message: changing the namespace of topics and adding the joint state publisher to the description launch file

File: fennec_description/urdf/fennec.xacro (robot description, xacro)
@@ -1,108 +1,129 @@
-<?xml version='1.0' ?>
-<robot name="jetracer" xmlns:xacro="http://www.ros.org/wiki/xacro">
-  <material name="black">
-    <color rgba="0 0 0 1"/>
-  </material>
-  <link name="base">
+<?xml version="1.0"?>
+<!--
+  Geometry:
+    The Ackermann steering controllers require the longitudinal
+    separation between the front and back wheel axes and the
+    lateral separation between the left and right front steering axes.
+    For this model:
+    wheel_separation_h = base_length - 2 * axle_offset = 0.4
+    wheel_separation_w = base_width  + 2 * axle_offset = 0.4
+-->
+<robot name="fennec" xmlns:xacro="http://wiki.ros.org/xacro">
+  <!-- Include xacro for inertials, materials and wheels -->
+  <xacro:include filename="$(find fennec_description)/urdf/wheel.xacro"/>
+  <!-- Gazebo plugins -->
+  <gazebo>
+    <plugin name="gazebo_ros_control" filename="libgazebo_ros_control.so">
+    </plugin>
+  </gazebo>
+  <!-- Math constants -->
+  <xacro:property name="deg_to_rad" value="0.01745329251994329577"/>
+  <!-- Robot base dimensions -->
+  <xacro:property name="base_length" value="0.34" />
+  <xacro:property name="base_width" value="0.16" />
+  <xacro:property name="base_height" value="0.16" />
+  <xacro:property name="base_mass" value="5" />
+  <!-- Wheel link dimensions -->
+  <xacro:property name="wheel_radius" value="0.034" />
+  <xacro:property name="wheel_thickness" value="0.025" />
+  <xacro:property name="wheel_mass" value="1" />
+  <!-- Steering link dimensions -->
+  <xacro:property name="steer_radius" value="0.05" />
+  <xacro:property name="steer_thickness" value="0.02" />
+  <xacro:property name="steer_mass" value="1" />
+  <!-- Axle positions -->
+  <xacro:property name="axle_offset" value="0.035" />
+  <xacro:property name="steer_offset" value="0.01" />
+  <!-- Base link -->
+  <link name="base_link">
     <visual>
-      <orgin rpy="0 0 0" xyz="0 0 0"/>
+      <origin xyz="0 0 0" rpy="0 0 0"/>
       <geometry>
-        <box size="1 2 0.3"/>
+        <box size="${base_length} ${base_width} ${base_height}"/>
       </geometry>
+      <material name="green" />
     </visual>
+    <collision>
+      <origin xyz="0 0 0" rpy="0 0 0"/>
+      <geometry>
+        <box size="${base_length} ${base_width} ${base_height}"/>
+      </geometry>
+    </collision>
+    <xacro:solid_cuboid_inertial
+        rpy="0 0 0" xyz="0 0 0"
+        mass="${base_mass}"
+        x="${base_length}" y="${base_width}" z="${base_height}" />
   </link>
-  <!--Front left wheel-->
-  <joint name="fl_holder_joint" type="revolute">
-    <axis xyz="0 0 1"/>
-    <limit effort="1000.0" lower="-0.4" upper="0.4" velocity="0.5"/>
-    <origin rpy="0 0 0" xyz="-0.5 0.8 0"/>
-    <parent link="base"/>
-    <child link="fl_wheel_link"/>
-  </joint>
-  <link name="fl_wheel_link">
-    <visual>
-      <orgin rpy="0 0 0" xyz="-0.7 0.8 0"/>
-      <geometry>
-        <box size="0 0 0"/>
-      </geometry>
-    </visual>
-  </link>
-  <joint name="fl_wheel_joint" type="continuous">
-    <axis xyz="0 0 1"/>
-    <origin rpy="0 1.57 0" xyz="-0.2 0 0"/>
-    <parent link="fl_wheel_link"/>
-    <child link="fl_wheel"/>
-  </joint>
-  <link name="fl_wheel">
-    <visual>
-      <orgin rpy="0 0 0" xyz="-0.7 0.8 0"/>
-      <geometry>
-        <cylinder radius="0.4" length="0.2"/>
-      </geometry>
-      <material name="black"/>
-    </visual>
-  </link>
-  <!--Front right wheel-->
-  <joint name="fr_holder_joint" type="revolute">
-    <axis xyz="0 0 1"/>
-    <limit effort="1000.0" lower="-0.4" upper="0.4" velocity="0.5"/>
-    <origin rpy="0 0 0" xyz="0.5 0.8 0"/>
-    <parent link="base"/>
-    <child link="fr_wheel_link"/>
-  </joint>
-  <link name="fr_wheel_link">
-    <visual>
-      <orgin rpy="0 0 0" xyz="0.7 0.8 0"/>
-      <geometry>
-        <box size="0 0 0"/>
-      </geometry>
-    </visual>
-  </link>
-  <joint name="fr_wheel_joint" type="continuous">
-    <axis xyz="0 0 1"/>
-    <origin rpy="0 1.57 0" xyz="0.2 0 0"/>
-    <parent link="fr_wheel_link"/>
-    <child link="fr_wheel"/>
-  </joint>
-  <link name="fr_wheel">
-    <visual>
-      <orgin rpy="0 0 0" xyz="0.7 0.8 0"/>
-      <geometry>
-        <cylinder radius="0.4" length="0.2"/>
-      </geometry>
-      <material name="black"/>
-    </visual>
-  </link>
-  <!--Rear left wheel-->
-  <joint name="rl_wheel_joint" type="continuous">
-    <axis xyz="0 0 1"/>
-    <origin rpy="0 1.57 0" xyz="-0.7 -0.8 0"/>
-    <parent link="base"/>
-    <child link="rl_wheel"/>
-  </joint>
-  <link name="rl_wheel">
-    <visual>
-      <orgin rpy="0 0 0" xyz="-0.7 -0.8 0"/>
-      <geometry>
-        <cylinder radius="0.4" length="0.2"/>
-      </geometry>
-      <material name="black"/>
-    </visual>
-  </link>
-  <!--Rear right wheel-->
-  <joint name="rr_wheel_joint" type="continuous">
-    <axis xyz="0 0 1"/>
-    <origin rpy="0 1.57 0" xyz="0.7 -0.8 0"/>
-    <parent link="base"/>
-    <child link="rr_wheel"/>
-  </joint>
-  <link name="rr_wheel">
-    <visual>
-      <orgin rpy="0 0 0" xyz="0.7 -0.8 0"/>
-      <geometry>
-        <cylinder radius="0.4" length="0.2"/>
-      </geometry>
-      <material name="black"/>
-    </visual>
-  </link>
+  <!-- Front steer and rear wheel joints required for ackermann_steering_controller -->
+  <xacro:rear_wheel
+    name="rear"
+    parent="base"
+    wheel_radius="${wheel_radius/4}"
+    wheel_thickness="${wheel_thickness/2}"
+    wheel_mass="${wheel_mass/32}">
+    <origin xyz="${-base_length/2+axle_offset} 0 0" rpy="${-90 * deg_to_rad} 0 0"/>
+  </xacro:rear_wheel>
+  <xacro:front_steer
+    name="front"
+    parent="base"
+    steer_radius="${steer_radius}"
+    steer_thickness="${steer_thickness}"
+    steer_mass="${steer_mass}"
+    base_length="${base_length}"
+    base_width="${base_width}"
+    axle_offset="${axle_offset}"
+    steer_height="${wheel_radius+steer_offset}">
+  </xacro:front_steer>
+  <!-- Rear wheels -->
+  <xacro:rear_wheel_lr
+    name="rear_right"
+    parent="base"
+    wheel_radius="${wheel_radius}"
+    wheel_thickness="${wheel_thickness}"
+    wheel_mass="${wheel_mass}">
+    <origin xyz="${-base_length/2+axle_offset} ${-base_width/2-axle_offset} 0" rpy="${-90 * deg_to_rad} 0 0"/>
+  </xacro:rear_wheel_lr>
+  <xacro:rear_wheel_lr
+    name="rear_left"
+    parent="base"
+    wheel_radius="${wheel_radius}"
+    wheel_thickness="${wheel_thickness}"
+    wheel_mass="${wheel_mass}">
+    <origin xyz="${-base_length/2+axle_offset} ${+base_width/2+axle_offset} 0" rpy="${-90 * deg_to_rad} 0 0"/>
+  </xacro:rear_wheel_lr>
+  <!-- Steerable front wheels -->
+  <xacro:front_wheel_lr
+    name="front_right"
+    parent="base"
+    reflect="-1"
+    wheel_radius="${wheel_radius}"
+    wheel_thickness="${wheel_thickness}"
+    wheel_mass="${wheel_mass}"
+    steer_radius="${steer_radius}"
+    steer_thickness="${steer_thickness}"
+    steer_mass="${steer_mass}"
+    base_length="${base_length}"
+    base_width="${base_width}"
+    axle_offset="${axle_offset}"
+    steer_height="${wheel_radius+steer_offset}">
+  </xacro:front_wheel_lr>
+  <xacro:front_wheel_lr
+    name="front_left"
+    parent="base"
+    reflect="1"
+    wheel_radius="${wheel_radius}"
+    wheel_thickness="${wheel_thickness}"
+    wheel_mass="${wheel_mass}"
+    steer_radius="${steer_radius}"
+    steer_thickness="${steer_thickness}"
+    steer_mass="${steer_mass}"
+    base_length="${base_length}"
+    base_width="${base_width}"
+    axle_offset="${axle_offset}"
+    steer_height="${wheel_radius+steer_offset}">
+  </xacro:front_wheel_lr>
+  <!-- Colour -->
+  <gazebo reference="base_link">
+    <material>Gazebo/Green</material>
+  </gazebo>
 </robot>

Commit message: Made it work

File: fennec_description/urdf/fennec.xacro (robot description, xacro)
@@ -22,5 +22,5 @@
   <xacro:property name="base_length" value="0.34" />
   <xacro:property name="base_width" value="0.16" />
-  <xacro:property name="base_height" value="0.16" />
+  <xacro:property name="base_height" value="0.08" />
   <xacro:property name="base_mass" value="5" />
   <!-- Wheel link dimensions -->
@@ -38,5 +38,5 @@
   <link name="base_link">
     <visual>
-      <origin xyz="0 0 0" rpy="0 0 0"/>
+      <origin xyz="0 0 0.06" rpy="0 0 0"/>
       <geometry>
         <box size="${base_length} ${base_width} ${base_height}"/>

File: fennec_description/urdf/wheel.xacro (robot description, xacro)
@@ -1,5 +1,5 @@
 <?xml version="1.0"?>
 <!--
-  Robot model adapted from https://github.com/CIR-KIT/steer_drive_ros/blob/kinetic-devel/steer_drive_controller/test/common/urdf/wheel.xacro
+  Robot model adapted from https://github.com/CIR-KI0.124T/steer_drive_ros/blob/kinetic-devel/steer_drive_controller/test/common/urdf/wheel.xacro
 -->
 <robot name="wheel" xmlns:xacro="http://wiki.ros.org/xacro">

Commit message: update to rviz visualization

File: fennec_description/urdf/fennec.xacro (robot description, xacro)
@@ -15,4 +15,5 @@
   <gazebo>
     <plugin name="gazebo_ros_control" filename="libgazebo_ros_control.so">
+      <robotNamespace>/fennec</robotNamespace>
     </plugin>
   </gazebo>
@@ -33,14 +34,15 @@
   <xacro:property name="steer_mass" value="1" />
   <!-- Axle positions -->
-  <xacro:property name="axle_offset" value="0.035" />
+  <xacro:property name="axle_offset" value="0.05" />
   <xacro:property name="steer_offset" value="0.01" />
   <!-- Base link -->
   <link name="base_link">
     <visual>
-      <origin xyz="0 0 0.06" rpy="0 0 0"/>
+      <origin xyz="0 0 0.05" rpy="0 0 1.57"/>
       <geometry>
-        <box size="${base_length} ${base_width} ${base_height}"/>
+        <!-- <box size="${base_length} ${base_width} ${base_height}"/>  0.0031 for stl -->
+        <mesh scale="0.0031 0.0031 0.0031" filename="package://fennec_description/meshes/fennec1.stl"/>
       </geometry>
-      <material name="green" />
+      <material name="white" />
     </visual>
     <collision>
@@ -82,5 +84,6 @@
     wheel_thickness="${wheel_thickness}"
     wheel_mass="${wheel_mass}">
-    <origin xyz="${-base_length/2+axle_offset} ${-base_width/2-axle_offset} 0" rpy="${-90 * deg_to_rad} 0 0"/>
+    <!-- <origin xyz="${-base_length/2+axle_offset} ${-base_width/2-axle_offset} 0" rpy="${-90 * deg_to_rad} 0 0"/> -->
+    <origin xyz="${-base_length/2+axle_offset} ${-base_width/2-axle_offset} 0" rpy="0 0 0"/>
   </xacro:rear_wheel_lr>
   <xacro:rear_wheel_lr
@@ -90,5 +93,6 @@
     wheel_thickness="${wheel_thickness}"
     wheel_mass="${wheel_mass}">
-    <origin xyz="${-base_length/2+axle_offset} ${+base_width/2+axle_offset} 0" rpy="${-90 * deg_to_rad} 0 0"/>
+    <!-- <origin xyz="${-base_length/2+axle_offset} ${+base_width/2+axle_offset} 0" rpy="${-90 * deg_to_rad} 0 0"/> -->
+    <origin xyz="${-base_length/2+axle_offset} ${+base_width/2+axle_offset} 0" rpy="0 0 0"/>
   </xacro:rear_wheel_lr>
   <!-- Steerable front wheels -->

File: fennec_description/urdf/wheel.xacro (robot description, xacro)
@@ -11,5 +11,5 @@
   <xacro:property name="steer_velocity" value="5.0"/>
   <xacro:property name="steer_limit_deg" value="45.0"/>
-  <!-- Bicycle model rear wheel link (required for steer_drive_controller) -->
+  <!-- Bicycle model rear wheel link (requiblack for steer_drive_controller) -->
   <xacro:macro name="rear_wheel"
     params="
@@ -25,6 +25,7 @@
         <geometry>
           <cylinder radius="${wheel_radius}" length="${wheel_thickness}"/>
-        </geometry>
-        <material name="yellow" />
+          <!-- <mesh scale="0.1 0.1 0.1" filename="package://fennec_description/meshes/dieciRear.stl"/> -->
+        </geometry>
+        <material name="black" />
       </visual>
       <collision>
@@ -48,5 +49,5 @@
       <type>transmission_interface/SimpleTransmission</type>
       <actuator name="${name}_wheel_joint_motor">
-        <mechanicalReduction>1</mechanicalReduction>
+        <mechanicalblackuction>1</mechanicalblackuction>
         <hardwareInterface>hardware_interface/VelocityJointInterface</hardwareInterface>
       </actuator>
@@ -59,6 +60,6 @@
     </gazebo>
   </xacro:macro>
-  <!-- Car steering model rear wheel links (left/right) -->
-  <xacro:macro name="rear_wheel_lr"
+  <!-- Bicycle model front wheel link (passive - no transmission) -->
+  <xacro:macro name="front_wheel"
     params="
       name
@@ -74,5 +75,5 @@
           <cylinder radius="${wheel_radius}" length="${wheel_thickness}"/>
         </geometry>
-        <material name="red" />
+        <material name="yellow" />
       </visual>
       <collision>
@@ -93,52 +94,4 @@
       <axis xyz="0 0 1"/>
     </joint>
-    <transmission name="${name}_wheel_joint_trans">
-      <type>transmission_interface/SimpleTransmission</type>
-      <actuator name="${name}_wheel_joint_motor">
-        <mechanicalReduction>1</mechanicalReduction>
-        <hardwareInterface>hardware_interface/VelocityJointInterface</hardwareInterface>
-      </actuator>
-      <joint name="${name}_wheel_joint">
-        <hardwareInterface>hardware_interface/VelocityJointInterface</hardwareInterface>
-      </joint>
-    </transmission>
-    <gazebo reference="${name}_wheel_link">
-      <material>Gazebo/Red</material>
-    </gazebo>
-  </xacro:macro>
-  <!-- Bicycle model front wheel link (passive - no transmission) -->
-  <xacro:macro name="front_wheel"
-    params="
-      name
-      parent
-      wheel_radius
-      wheel_thickness
-      wheel_mass
-      *origin">
-    <link name="${name}_wheel_link">
-      <visual>
-        <origin xyz="0 0 0" rpy="0 0 0"/>
-        <geometry>
-          <cylinder radius="${wheel_radius}" length="${wheel_thickness}"/>
-        </geometry>
-        <material name="yellow" />
-      </visual>
-      <collision>
-        <origin xyz="0 0 0" rpy="0 0 0"/>
-        <geometry>
-          <cylinder radius="${wheel_radius}" length="${wheel_thickness}"/>
-        </geometry>
-      </collision>
-      <xacro:solid_cylinder_inertial
-          rpy="0 0 0" xyz="0 0 0"
-          mass="${wheel_mass}"
-          radius="${wheel_radius}" length="${wheel_thickness}" />
-    </link>
-    <joint name="${name}_wheel_joint" type="continuous">
-      <parent link="${parent}_link"/>
-      <child link="${name}_wheel_link"/>
-      <xacro:insert_block name="origin"/>
-      <axis xyz="0 0 1"/>
-    </joint>
     <gazebo reference="${name}_wheel_link">
       <material>Gazebo/Yellow</material>
@@ -148,5 +101,5 @@
     </gazebo>
   </xacro:macro>
-  <!-- Bicycle model front steering link (required for steer_drive_controller) -->
+  <!-- Bicycle model front steering link (requiblack for steer_drive_controller) -->
   <xacro:macro name="front_steer"
     params="
@@ -161,5 +114,5 @@
       steer_height">
     <link name="${name}_steer_link">
-      <visual>
+      <!-- <visual>
         <origin xyz="0 0 0" rpy="0 0 0"/>
         <geometry>
@@ -167,5 +120,5 @@
         </geometry>
         <material name="yellow" />
-      </visual>
+      </visual> -->
       <collision>
         <origin xyz="0 0 0" rpy="0 0 0"/>
@@ -191,5 +144,5 @@
       <type>transmission_interface/SimpleTransmission</type>
       <actuator name="${name}_steer_joint_motor">
-        <mechanicalReduction>1</mechanicalReduction>
+        <mechanicalblackuction>1</mechanicalblackuction>
         <hardwareInterface>hardware_interface/PositionJointInterface</hardwareInterface>
       </actuator>
@@ -200,4 +153,53 @@
     <gazebo reference="${name}_steer_link">
       <material>Gazebo/Yellow</material>
+    </gazebo>
+  </xacro:macro>
+  <!-- Car steering model rear wheel links (left/right) -->
+  <xacro:macro name="rear_wheel_lr"
+    params="
+      name
+      parent
+      wheel_radius
+      wheel_thickness
+      wheel_mass
+      *origin">
+    <link name="${name}_wheel_link">
+      <visual>
+        <origin xyz="0 0 0" rpy="0 0 0"/>
+        <geometry>
+          <!-- <cylinder radius="${wheel_radius}" length="${wheel_thickness}"/> -->
+          <mesh scale="0.0025 0.0025 0.0025" filename="package://fennec_description/meshes/dieciRear.stl"/>
+        </geometry>
+        <material name="black" />
+      </visual>
+      <collision>
+        <origin xyz="0 0 0" rpy="0 0 0"/>
+        <geometry>
+          <cylinder radius="${wheel_radius}" length="${wheel_thickness}"/>
+        </geometry>
+      </collision>
+      <xacro:solid_cylinder_inertial
+          rpy="0 0 0" xyz="0 0 0"
+          mass="${wheel_mass}"
+          radius="${wheel_radius}" length="${wheel_thickness}" />
+    </link>
+    <joint name="${name}_wheel_joint" type="continuous">
+      <parent link="${parent}_link"/>
+      <child link="${name}_wheel_link"/>
+      <xacro:insert_block name="origin"/>
+      <axis xyz="0 0 1"/>
+    </joint>
+    <transmission name="${name}_wheel_joint_trans">
+      <type>transmission_interface/SimpleTransmission</type>
+      <actuator name="${name}_wheel_joint_motor">
+        <mechanicalblackuction>1</mechanicalblackuction>
+        <hardwareInterface>hardware_interface/VelocityJointInterface</hardwareInterface>
+      </actuator>
+      <joint name="${name}_wheel_joint">
+        <hardwareInterface>hardware_interface/VelocityJointInterface</hardwareInterface>
+      </joint>
+    </transmission>
+    <gazebo reference="${name}_wheel_link">
+      <material>Gazebo/black</material>
     </gazebo>
   </xacro:macro>
@@ -219,5 +221,5 @@
       steer_height">
     <link name="${name}_steer_link">
-      <visual>
+      <!-- <visual>
         <origin xyz="0 0 0" rpy="0 0 0"/>
         <geometry>
@@ -225,5 +227,5 @@
         </geometry>
         <material name="blue" />
-      </visual>
+      </visual> -->
       <collision>
         <origin xyz="0 0 0" rpy="0 0 0"/>
@@ -250,7 +252,8 @@
         <origin xyz="0 0 0" rpy="0 0 0"/>
         <geometry>
-          <cylinder radius="${wheel_radius}" length="${wheel_thickness}"/>
-        </geometry>
-        <material name="red" />
+          <!-- <cylinder radius="${wheel_radius}" length="${wheel_thickness}"/> -->
+          <mesh scale="0.0022 0.0022 0.0022" filename="package://fennec_description/meshes/dieciRear.stl"/>
+        </geometry>
+        <material name="black" />
       </visual>
       <collision>
@@ -274,5 +277,5 @@
       <type>transmission_interface/SimpleTransmission</type>
       <actuator name="${name}_steer_joint_motor">
-        <mechanicalReduction>1</mechanicalReduction>
+        <mechanicalblackuction>1</mechanicalblackuction>
         <hardwareInterface>hardware_interface/PositionJointInterface</hardwareInterface>
       </actuator>
@@ -284,5 +287,5 @@
       <type>transmission_interface/SimpleTransmission</type>
       <actuator name="${name}_wheel_joint_motor">
-        <mechanicalReduction>1</mechanicalReduction>
+        <mechanicalblackuction>1</mechanicalblackuction>
         <hardwareInterface>hardware_interface/VelocityJointInterface</hardwareInterface>
       </actuator>
@@ -295,5 +298,5 @@
     </gazebo>
     <gazebo reference="${name}_wheel_link">
-      <material>Gazebo/Red</material>
+      <material>Gazebo/black</material>
     </gazebo>
   </xacro:macro>
